File: PCB_TFG/PCB_TFG.kicad_pcb (KiCad board)
At the start: 2 copper layers, 134.2 x 61.5 mm, 21 parts, among them J1 JST, J2 TFT_Pantalla, J3 Joystick1, J4 Joystick2, SW1 Switch1, SW2 Switch2, SW3 Switch3, SW4 Switch4, SW5 Switch5, SW6 Switch6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

Commit message: Actualización Interruptor
Parts:
- SW8: value Interruptor -> SW_SPDT; footprint Button_Switch_THT:SW_DIP_SPSTx01_Slide_6.7x4.1mm_W7.62mm_P2.54mm_LowProfile -> Button_Switch_THT:SW_Slide-03_Wuerth-WS-SLTV_10x2.5x6.4_P2.54mm
- moved SW8 4.40 mm to (179.2, 77.0), turned to 90 degrees
Connections:
- SW8 pad 1: Net-(SW8B-C) -> GND
- SW8 pad 2: Net-(SW8B-D) -> Net-(SW8-B)
- TP1 pad 5: Net-(SW8B-C) -> Net-(SW8-B)
- U3 pad 1: Net-(SW8B-D) -> Net-(SW8-C)
Routing:
- net Net-(SW8-C): track 0.00 -> 44.4 mm
- net Net-(SW8B-D): track 38.9 -> 0.00 mm
- net Net-(SW8B-C): track 36.5 -> 0.00 mm
- net Net-(SW8-B): track 0.00 -> 28.4 mm
